File: opticore/EAGLE/core.sch (EAGLE design)
At the start: 35 parts, among them IC1 LM2596T, J1 POWER_JACKSLT, T1 TRIACPTH, T2 TRIACPTH, T3 TRIACPTH, T4 TRIACPTH, T5 TRIACPTH, T6 TRIACPTH, T7 TRIACPTH, T8 TRIACPTH, X1 FFKV8

Commit message: Adding BOM
Idk what the board updates are.
Parts:
- C1, C2, C3: MPN (none) -> 10NA100MEFC6.3X11; OC_NEWARK (none) -> 54T4154
- C4, C5, H1, H2, J1, JP10, JP11, JP12, LOGO2, SJ1, U$3: OC_NEWARK (none) -> unknown
- COM: MPN (none) -> 724; OC_NEWARK (none) -> 53W6206
- D1, D2: MF (none) -> FAIRCHILD SEMICONDUCTOR; MPN (none) -> 1N4004; OC_NEWARK (none) -> 18C8917
- D3: MPN (none) -> L-710A8CB/1GD; OC_NEWARK (none) -> 87W9956
- IC1: MF (none) -> NATIONAL SEMICONDUCTOR; MPN (none) -> LM2596T-5.0/NOPB; OC_NEWARK (none) -> 41K3851
- IC2: MPN (none) -> LM1117MPX-3.3/NOPB; OC_NEWARK (none) -> 12X9029
- L1: MPN (none) -> RLB9012-151KL; OC_NEWARK (none) -> 32M9853
- R1: MF (none) -> FARNELL; MPN (none) -> MCF 1W 1K; OC_NEWARK (none) -> 38K0400
- R2, R3: MF (none) -> FARNELL; MPN (none) -> MF25 4K7; OC_NEWARK (none) -> 38K5355
- RN1, RN2: MPN (none) -> CSC09A01330RGEK; OC_NEWARK (none) -> 71M1507
- T1, T2, T3, T4, T5, T6, T7, T8: MF (none) -> ON SEMICONDUCTOR; MPN (none) -> MAC97A6G; OC_NEWARK (none) -> 26K3660
